Commit message: Update joint parameters in alpha.urdf.xacro for improved kinematics

File: ReachAlpha5/alpha_description/urdf/alpha.urdf.xacro (robot description, xacro)
@@ -108,7 +108,7 @@
       <parent link="${prefix}m2_1_1_link" />
       <child link="${prefix}m2_joint_link" />
-      <origin xyz="-0.02 0 0.033" />
+      <origin xyz="-0.02 0 0.033" rpy="0.0 -1.571 0.0" />
       <axis xyz="0 1 0" />
-      <limit effort="9.0" lower="0.0" upper="3.49" velocity="0.5" />
+      <limit effort="9.0" lower="1.571" upper="4.713" velocity="0.5" />
     </joint>
     <link name="${prefix}m2_1_2_link">

Commit message: Add mounting plate link and joint to alpha.urdf.xacro for enhanced structure

File: ReachAlpha5/alpha_description/urdf/alpha.urdf.xacro (robot description, xacro)
@@ -12,4 +12,26 @@
     </material>
     <link name="${prefix}base_link" />
+    <link name="${prefix}mounting_plate">
+      <inertial>
+        <origin xyz="0.0 -0.0096 0.0045" rpy="0 0 0"/>
+        <mass value="0.20062240239642046"/>
+        <inertia ixx="8.1e-05" iyy="9.5e-05" izz="5.4e-05" ixy="0.0" iyz="1.6e-05" ixz="0.0"/>
+      </inertial>
+      <visual>
+        <origin xyz="0.0 0.0 0.0" rpy="0 0 0"/>
+        <geometry>
+          <mesh filename="file://$(find alpha_description)/meshes/mounting_plate_1.stl" scale="0.001 0.001 0.001"/>
+        </geometry>
+        <material name="opaque157207237">
+          <color rgba="0.6156 0.8117 0.9294 1.0"/>
+        </material>
+      </visual>
+      <collision>
+        <origin xyz="0.0 0.0 0.0" rpy="0 0 0"/>
+        <geometry>
+          <mesh filename="file://$(find alpha_description)/meshes/mounting_plate_1.stl" scale="0.001 0.001 0.001"/>
+        </geometry>
+      </collision>
+    </link>
     <link name="${prefix}m3_inline_link">
       <visual>
@@ -29,14 +51,16 @@
         <mass value="0.341" />
         <origin xyz="-0.075 -0.006 -0.003" />
-        <inertia
-          ixx="0.000099" ixy="0.000139" ixz="0.000115"
-          iyx="0.000139" iyy="0.00292" iyz="0.000003"
-          izx="0.000115" izy="0.000003" izz="0.002934" />
+        <inertia ixx="0.000099" ixy="0.000139" ixz="0.000115" iyx="0.000139" iyy="0.00292" iyz="0.000003" izx="0.000115" izy="0.000003" izz="0.002934" />
       </inertial>
     </link>
     <joint name="${prefix}base_link_joint" type="fixed">
       <parent link="${prefix}base_link" />
+      <child link="${prefix}mounting_plate" />
+      <origin rpy="0 0 0" />
+    </joint>
+    <joint name="${prefix}mounting_plate_joint" type="fixed">
+      <parent link="${prefix}mounting_plate" />
       <child link="${prefix}m3_inline_link" />
-      <origin rpy="0 0 0" />
+      <origin xyz="0 -0.025 0.037" />
     </joint>
     <link name="${prefix}m2_1_1_link">
@@ -57,8 +81,5 @@
         <mass value="0.194" />
         <origin xyz="0.005 -0.001 0.016" />
-        <inertia
-          ixx="0.000189" ixy="0.000005" ixz="0.000054"
-          iyx="0.000005" iyy="0.000213" iyz="0.000003"
-          izx="0.000054" izy="0.000003" izz="0.000067" />
+        <inertia ixx="0.000189" ixy="0.000005" ixz="0.000054" iyx="0.000005" iyy="0.000213" iyz="0.000003" izx="0.000054" izy="0.000003" izz="0.000067" />
       </inertial>
     </link>
@@ -66,5 +87,6 @@
       <parent link="${prefix}m3_inline_link" />
       <child link="${prefix}m2_1_1_link" />
-      <origin xyz="0 0 0.014" />
+      <!-- <origin xyz="0 0 0.014" /> -->
+      <origin xyz="0 0 0.15" rpy="0 -1.571 0"/>
       <axis xyz="0 0 1" />
       <limit effort="9.0" lower="0.0" upper="6.10" velocity="0.5" />
@@ -99,8 +121,5 @@
         <mass value="0.429" />
         <origin xyz="0.073 0.0 0.0" />
-        <inertia
-          ixx="0.000087" ixy="-0.000076" ixz="-0.00001"
-          iyx="-0.000076" iyy="0.00319" iyz="0"
-          izx="-0.00001" izy="0" izz="0.003212" />
+        <inertia ixx="0.000087" ixy="-0.000076" ixz="-0.00001" iyx="-0.000076" iyy="0.00319" iyz="0" izx="-0.00001" izy="0" izz="0.003212" />
       </inertial>
     </link>
@@ -108,5 +127,5 @@
       <parent link="${prefix}m2_1_1_link" />
       <child link="${prefix}m2_joint_link" />
-      <origin xyz="-0.02 0 0.033" rpy="0.0 -1.571 0.0" />
+      <origin xyz="-0.02 0 0.033" rpy="0.0 0.0 0.0" />
       <axis xyz="0 1 0" />
       <limit effort="9.0" lower="1.571" upper="4.713" velocity="0.5" />
@@ -129,8 +148,5 @@
         <mass value="0.115" />
         <origin xyz="0.017 -0.026 -0.002" />
-        <inertia
-          ixx="0.00012" ixy="-0.000061" ixz="-0.000001"
-          iyx="-0.000061" iyy="0.000062" iyz="0"
-          izx="-0.000001" izy="0" izz="0.000156" />
+        <inertia ixx="0.00012" ixy="-0.000061" ixz="-0.000001" iyx="-0.000061" iyy="0.000062" iyz="0" izx="-0.000001" izy="0" izz="0.000156" />
       </inertial>
     </link>
@@ -145,6 +161,5 @@
       <visual>
         <geometry>
-          <mesh
-            filename="file://$(find alpha_description)/meshes/RS1-100-101-123.stl" />
+          <mesh filename="file://$(find alpha_description)/meshes/RS1-100-101-123.stl" />
         </geometry>
         <origin rpy="0 -1.5707 0" xyz="0 0 0" />
@@ -160,8 +175,5 @@
         <mass value="0.333" />
         <origin xyz="0.0 0.003 -0.098" />
-        <inertia
-          ixx="0.003709" ixy="0.000002" ixz="-0.000004"
-          iyx="0.000002" iyy="0.003734" iyz="0"
-          izx="-0.000004" izy="0" izz="0.000079" />
+        <inertia ixx="0.003709" ixy="0.000002" ixz="-0.000004" iyx="0.000002" iyy="0.003734" iyz="0" izx="-0.000004" izy="0" izz="0.000079" />
       </inertial>
     </link>
@@ -184,6 +196,5 @@
       <inertial>
         <mass value="2e-06" />
-        <inertia ixx="1.1e-09" ixy="0" ixz="0" iyy="1.1e-09" iyz="0"
-          izz="1.1e-09" />
+        <inertia ixx="1.1e-09" ixy="0" ixz="0" iyy="1.1e-09" iyz="0" izz="1.1e-09" />
       </inertial>
     </link>
@@ -191,6 +202,5 @@
       <inertial>
         <mass value="2e-06" />
-        <inertia ixx="1.1e-09" ixy="0" ixz="0" iyy="1.1e-09" iyz="0"
-          izz="1.1e-09" />
+        <inertia ixx="1.1e-09" ixy="0" ixz="0" iyy="1.1e-09" iyz="0" izz="1.1e-09" />
       </inertial>
     </link>
@@ -202,9 +212,6 @@
       <limit effort="10" lower="0" upper="0.015" velocity="10" />
     </joint>
-    <xacro:include
-      filename="$(find alpha_description)/urdf/end_effectors/standard_jaws.urdf.xacro" />
-    <xacro:alpha_standard_jaws parent="${prefix}ee_base_link"
-      prefix="${prefix}standard_jaws_"
-      axis_a="${prefix}axis_a">
+    <xacro:include filename="$(find alpha_description)/urdf/end_effectors/standard_jaws.urdf.xacro" />
+    <xacro:alpha_standard_jaws parent="${prefix}ee_base_link" prefix="${prefix}standard_jaws_" axis_a="${prefix}axis_a">
       <origin xyz="0 0 0" rpy="0 0 0" />
     </xacro:alpha_standard_jaws>

Commit message: Refactor joint origins and collision geometry in alpha.urdf.xacro for improved accuracy

File: ReachAlpha5/alpha_description/urdf/alpha.urdf.xacro (robot description, xacro)
@@ -39,12 +39,16 @@
           <mesh filename="file://$(find alpha_description)/meshes/M3-INLINE.stl" />
         </geometry>
-        <origin rpy="0 0 0" xyz="0 0 0" />
-        <material name="${prefix}black" />
-      </visual>
-      <collision>
-        <geometry>
+        <origin rpy="0 -1.57075 0" xyz="0.0 0.004 0.1225" />
+        <material name="${prefix}black" />
+      </visual>
+      <collision>
+        <!-- <geometry>
           <cylinder length="0.150" radius="0.020" />
         </geometry>
-        <origin rpy="0 1.57075 0" xyz="-0.075 0 0" />
+        <origin rpy="0 1.57075 0" xyz="-0.075 0 0" /> -->
+        <geometry>
+          <mesh filename="file://$(find alpha_description)/meshes/M3-INLINE.stl" />
+        </geometry>
+        <origin rpy="0 -1.57075 0" xyz="0.0 0.004 0.1225" />
       </collision>
       <inertial>
@@ -62,5 +66,5 @@
       <parent link="${prefix}mounting_plate" />
       <child link="${prefix}m3_inline_link" />
-      <origin xyz="0 -0.025 0.037" />
+      <origin xyz="0.0 -0.025 0.037" rpy="0 0 -1.57075"/>
     </joint>
     <link name="${prefix}m2_1_1_link">
@@ -88,7 +92,8 @@
       <child link="${prefix}m2_1_1_link" />
       <!-- <origin xyz="0 0 0.014" /> -->
-      <origin xyz="0 0 0.15" rpy="0 -1.571 0"/>
+      <origin xyz="-0.0135 0.005 0.1225" rpy="0 1.57075 3.142"/>
       <axis xyz="0 0 1" />
-      <limit effort="9.0" lower="0.0" upper="6.10" velocity="0.5" />
+      <!-- <limit effort="9.0" lower="0.0" upper="6.10" velocity="0.5" /> -->
+      <limit effort="9.0" lower="-3.142" upper="3.142" velocity="0.5" />
     </joint>
     <link name="${prefix}m2_joint_link">
@@ -127,5 +132,6 @@
       <parent link="${prefix}m2_1_1_link" />
       <child link="${prefix}m2_joint_link" />
-      <origin xyz="-0.02 0 0.033" rpy="0.0 0.0 0.0" />
+      <!-- <origin xyz="-0.02 0 0.033" rpy="0.0 0.0 0.0" /> -->
+      <origin xyz="-0.02 0 0.033" rpy="0.0 0.0 3.142" />
       <axis xyz="0 1 0" />
       <limit effort="9.0" lower="1.571" upper="4.713" velocity="0.5" />
